File: DonkeyHat/_autosave-DonkeyHat.kicad_sch (KiCad schematic)
At the start: 11 parts, among them J1 GPIO, J2 Conn_01x02_Pin, U1 ProMicro

Commit message: Switched to smaller 2040
Parts:
- renumbered J2 to 5V, Encoder to Encoder1
Changed lines of the file:
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@@
 		(dnp no)
 		(fields_autoplaced yes)
-		(property "Reference" "Encoder"
+		(property "Reference" "Encoder1"
 			(at 38.735 82.55 0)
 			(effects
@@
 			(project "DonkeyHat"
 				(path "/e63e39d7-6ac0-4ffd-8aa3-1841a4541b55"
-					(reference "Encoder")
+					(reference "Encoder1")
 					(unit 1)
 				)
@@
 		(dnp no)
 		(fields_autoplaced yes)
-		(property "Reference" "J2"
+		(property "Reference" "5V"
 			(at 88.9 16.5099 0)
 			(effects
@@
 			(project "DonkeyHat"
 				(path "/e63e39d7-6ac0-4ffd-8aa3-1841a4541b55"
-					(reference "J2")
+					(reference "5V")
 					(unit 1)
 				)
