File: DonkeyHat/DonkeyHatZero.kicad_pcb (KiCad board)
At the start: 2 copper layers, 65 x 29.2 mm, 9 parts, among them J1 GPIO, J4 I2C, U2 rp2040-zero

Commit message: Zero WIP
Parts:
- removed 5V1: Conn_01x02_Pin, Connector_PinHeader_2.54mm:PinHeader_1x02_P2.54mm_Vertical
- removed I2C1, OLED1: Conn_01x04_Pin, Connector_PinHeader_2.54mm:PinHeader_1x04_P2.54mm_Vertical
- removed J4: I2C, Connector_JST:JST_SH_BM04B-SRSS-TB_1x04-1MP_P1.00mm_Vertical
- added J2: Conn_01x02_Pin, Connector_PinHeader_2.54mm:PinHeader_1x02_P2.54mm_Vertical, F.Cu at (163.5, 56.8)
- added J3: Conn_01x02_Pin, Connector_PinHeader_2.54mm:PinHeader_1x02_P2.54mm_Vertical, F.Cu at (163.5, 67.0)
- added J5: Battery +, Connector_PinHeader_2.54mm:PinHeader_1x01_P2.54mm_Vertical, B.Cu at (158.4, 56.8)
- added J6: Battery -, Connector_PinHeader_2.54mm:PinHeader_1x01_P2.54mm_Vertical, B.Cu at (150.8, 56.8)
- added J7: +5v, Connector_PinHeader_2.54mm:PinHeader_1x01_P2.54mm_Vertical, B.Cu at (150.8, 67.7)
- added J8: GND, Connector_PinHeader_2.54mm:PinHeader_1x01_P2.54mm_Vertical, B.Cu at (158.4, 68.0)
- added Steer1: Conn_01x03_Pin, Connector_PinHeader_2.54mm:PinHeader_1x03_P2.54mm_Vertical, F.Cu at (102.0, 65.5)
- U2: moved to B.Cu
- moved RCin1 61.9 mm to (102.1, 54.7), turned to 0 degrees
- moved U2 4.56 mm to (117.4, 63.1), turned to -90 degrees
- renumbered Throttle1 to RCin1
Connections:
- J1 pad 1: +3V3 -> unconnected-(J1-Pin_1-Pad1)
- J1 pad 17: +3V3 -> unconnected-(J1-Pin_17-Pad17)
- J1 pad 20: GND -> unconnected-(J1-Pin_20-Pad20)
- J1 pad 25: GND -> unconnected-(J1-Pin_25-Pad25)
- J1 pad 29: /GPIO5 -> unconnected-(J1-Pin_29-Pad29)
- J1 pad 3: /GPIO2/SDA1 -> unconnected-(J1-Pin_3-Pad3)
- J1 pad 30: GND -> unconnected-(J1-Pin_30-Pad30)
- J1 pad 34: GND -> unconnected-(J1-Pin_34-Pad34)
- J1 pad 39: GND -> unconnected-(J1-Pin_39-Pad39)
- J1 pad 5: /GPIO3/SCL1 -> unconnected-(J1-Pin_5-Pad5)
- J1 pad 9: GND -> unconnected-(J1-Pin_9-Pad9)
- RCin1 pad 2: +5V -> Batt
- RCin1 pad 3: RCin3 -> RCin1
- U2 pad 11: Throttle -> unconnected-(U2-10-Pad11)
- U2 pad 17: RCin2 -> unconnected-(U2-26-Pad17)
- U2 pad 20: RCin3 -> unconnected-(U2-29-Pad20)
Other:
- board size 65 x 29.2 mm -> 66.2 x 29.2 mm
- board text removed: "- +"
- board text removed: "- + SCL SDA"
- board text removed: "5V"
- board text removed: "I2C"

Commit message: Ready for routing
Parts:
- moved J8 8.42 mm to (150.0, 68.0)
- moved J7 7.71 mm to (158.5, 68.0)
- moved J6 0.80 mm to (150.0, 56.8)
Other:
- board text added: "- +"
- board text added: "Batt"
- board text added: "Car"
Changed lines of the file:
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@@
 	(footprint "Connector_PinHeader_2.54mm:PinHeader_1x01_P2.54mm_Vertical"
 		(layer "B.Cu")
-		(at 158.42 67.95)
+		(at 150 68)
 		(descr "Through hole straight pin header, 1x01, 2.54mm pitch, single row")
 		(tags "Through hole pin header THT 1x01 2.54mm single row")
@@
 	(footprint "Connector_PinHeader_2.54mm:PinHeader_1x01_P2.54mm_Vertical"
 		(layer "B.Cu")
-		(at 150.8 56.82)
+		(at 150 56.82)
 		(descr "Through hole straight pin header, 1x01, 2.54mm pitch, single row")
 		(tags "Through hole pin header THT 1x01 2.54mm single row")
@@
 	(footprint "Connector_PinHeader_2.54mm:PinHeader_1x01_P2.54mm_Vertical"
 		(layer "B.Cu")
-		(at 150.8 67.69)
+		(at 158.5 68)
 		(descr "Through hole straight pin header, 1x01, 2.54mm pitch, single row")
 		(tags "Through hole pin header THT 1x01 2.54mm single row")
@@
 		)
 	)
+	(gr_text "Batt"
+		(at 160.9 59.5 90)
+		(layer "F.SilkS")
+		(effects
+			(font
+				(size 1 1)
+				(thickness 0.15)
+			)
+			(justify left bottom)
+		)
+	)
 	(gr_text "S  +  -"
 		(at 105.55 60.58 90)
@@
 			)
 			(justify left bottom)
+		)
+	)
+	(gr_text "-   +"
+		(at 161.6 60.3 90)
+		(layer "F.SilkS")
+		(effects
+			(font
+				(size 1 1)
+				(thickness 0.15)
+			)
+			(justify left bottom)
+		)
+	)
+	(gr_text "Car"
+		(at 161 69.4 90)
+		(layer "F.SilkS")
+		(effects
+			(font
+				(size 1 1)
+				(thickness 0.15)
+			)
+			(justify left bottom)
+		)
+	)
+	(gr_text "-   +"
+		(at 161.6 70.6 90)
+		(layer "F.SilkS")
+		(effects
+			(font
+				(size 1 1)
+				(thickness 0.15)
+			)
+			(justify left bottom)
